File: Insignis/Connectors.kicad_sch (KiCad schematic)
At the start: 30 parts, among them J1 Conn_Coaxial, J10 USB_JST, J11 PT_1, J12 FILL, J2 Conn_Coaxial, J3 USB_C_Receptacle, J4 Switch, J5 PWR, J6 PT_2, J7 PT_3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

Commit message: Fixed ERC errors
Parts:
- J10: footprint SM04B-GHS-TB -> SM04B-GHS-TB_LF__SN_:SM04B-GHS-TB
- J11, J12, J6, J7, J9: footprint SM02BGHSTBLFSN -> SM02B-GHS-TB_LF__SN_:SM02BGHSTBLFSN
- J5: footprint S2BPHSM4TBLFSN -> S2B-PH-SM4-TB_LF__SN_:S2BPHSM4TBLFSN
- J8: footprint S3BPHSM4TBLFSN -> S3B-PH-SM4-TB_LF__SN_:S3BPHSM4TBLFSN
- Q1: footprint SOT95P280X125-3N -> AO3401A:SOT95P280X125-3N
- Q2: footprint SOT95P240X120-3N -> BSS138:SOT95P240X120-3N
