File: Insignis/Indication.kicad_sch (KiCad schematic)
At the start: 6 parts

Commit message: Fixed ERC errors
Parts:
- LED1: footprint LRTB-R48G -> LRTB_R48G:LRTB-R48G
- LS1: footprint CPT9019ASMTTR -> CPT-9019A-SMT-TR:CPT9019ASMTTR
Changed lines of the file:
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@@
 			)
 		)
-		(property "Description" ""
+		(property "Description" "Power symbol creates a global label with name \"GND\" , ground"
 			(at 138.43 99.06 0)
 			(effects
@@
 					(size 1.27 1.27)
 				)
+				(hide yes)
 			)
 		)
@@
 			)
 		)
-		(property "Footprint" "CPT9019ASMTTR"
+		(property "Footprint" "CPT-9019A-SMT-TR:CPT9019ASMTTR"
 			(at 152.4 196.52 0)
 			(effects
@@
 			)
 		)
-		(property "Description" ""
+		(property "Description" "Power symbol creates a global label with name \"+3V3\""
 			(at 171.45 67.31 0)
 			(effects
@@
 					(size 1.27 1.27)
 				)
+				(hide yes)
 			)
 		)
@@
 			)
 		)
-		(property "Footprint" "LRTB-R48G"
+		(property "Footprint" "LRTB_R48G:LRTB-R48G"
 			(at 161.29 164.77 0)
 			(effects
